File: micro_rusEFI.sch (KiCad schematic (older format))
At the start: 57 parts, among them J12 Conn_01x01, J13 Conn_01x01, J3 Conn_01x01, J4 Conn_02x05_Counter_Clockwise, J5 Conn_01x01, U3 molex_48pin_MRE, U7 XC6206 3.3V

Commit message: Add files via upload
Parts:
- added D44: B5819W, Diode_SMD:D_SOD-123, symbol micro_rusEFI-rescue:D_Schottky-Device
- added JP3: Voltage selector 5V 3V3, Jumper:SolderJumper-3_P1.3mm_Bridged12_RoundedPad1.0x1.5mm, symbol micro_rusEFI-rescue:SolderJumper_3_Open-Jumper
- added unit 18 of U3
- added unit 17 of U3
- D15, D20, D3, D4, D5, D6, D7: symbol Device:D_Schottky -> micro_rusEFI-rescue:D_Schottky-Device
- D21, D22, D23, D27, D28, D31, D33, D35: symbol Device:LED -> micro_rusEFI-rescue:LED-Device
- D30, D32, D34, D43: symbol Device:D -> micro_rusEFI-rescue:D-Device
- D36, D37: footprint Diode_SMD:D_SMA -> Diode_SMD:D_SMC; symbol Diode:B340 -> micro_rusEFI-rescue:B340-Diode
- D41: symbol Device:D_TVS -> micro_rusEFI-rescue:D_TVS-Device
- J12, J13, J3, J5: symbol Connector_Generic:Conn_01x01 -> micro_rusEFI-rescue:Conn_01x01-Connector_Generic
- J4: symbol Connector_Generic:Conn_02x05_Odd_Even -> micro_rusEFI-rescue:Conn_02x05_Odd_Even-Connector_Generic
- LOGO1: symbol Graphic:Logo_Open_Hardware_Small -> micro_rusEFI-rescue:Logo_Open_Hardware_Small-Graphic
- NT2, NT3: symbol Device:Net-Tie_2 -> micro_rusEFI-rescue:Net-Tie_2-Device
- R10, R2, R21, R29, R30, R33, R36, R49, R51, R80, R81, R84, R85, R86: symbol Device:R -> micro_rusEFI-rescue:R-Device
- RN1: symbol Device:R_Pack04 -> micro_rusEFI-rescue:R_Pack04-Device
- TP0, TP1, TP12, TP2, TP3, TP4, TP5: symbol Connector:TestPoint -> micro_rusEFI-rescue:TestPoint-Connector
- U3: footprint rusefi_lib:Molex_48_MRE -> rusefi_lib:Molex_48_MRE_R055; symbol rusefi_Molex_MRE_Connector:molex_48pin_MRE -> micro_rusEFI-rescue:molex_48pin_MRE-rusefi_Molex_MRE_Connector
- U7: symbol Regulator_Linear:MCP1703A-3302_SOT23 -> micro_rusEFI-rescue:MCP1703A-3302_SOT23-Regulator_Linear
Connections:
- wire segments 325 -> 335
