File: micro_rusEFI.sch (KiCad schematic (older format))
At the start: 59 parts, among them J12 Conn_01x01, J13 Conn_01x01, J3 Conn_01x01, J4 Conn_02x05_Counter_Clockwise, J5 Conn_01x01, U3 molex_48pin_MRE, U7 XC6206 3.3V

Commit message: Add files via upload
Parts:
- D36, D37: footprint Diode_SMD:D_SMC -> Diode_SMD:D_SMA
Changed lines of the file:
@@
 Sheet 1 10
 Title "microRusEFI-2L"
-Date "2021-12-29"
+Date "2021-12-30"
 Rev "R0.5.5rc2"
 Comp "rusEFI.com"
@@
 F 0 "D36" H 11275 1675 50  0000 C CNN
 F 1 "SS54" H 11275 1875 50  0000 C CNN
-F 2 "Diode_SMD:D_SMC" H 11275 1600 50  0001 C CNN
+F 2 "Diode_SMD:D_SMA" H 11275 1600 50  0001 C CNN
 F 3 "" H 11275 1775 50  0001 C CNN
 F 4 "C22452" H 11275 1775 50  0001 C CNN "LCSC"
@@
 F 0 "D37" H 11275 2050 50  0000 C CNN
 F 1 "SS54" H 11275 2250 50  0000 C CNN
-F 2 "Diode_SMD:D_SMC" H 11275 1975 50  0001 C CNN
+F 2 "Diode_SMD:D_SMA" H 11275 1975 50  0001 C CNN
 F 3 "" H 11275 2150 50  0001 C CNN
 F 4 "C22452" H 11275 2150 50  0001 C CNN "LCSC"
@@
 	1    0    0    -1
 $EndComp
-$Comp
-L micro_rusEFI-rescue:D_Schottky-Device D44
-U 1 1 618B2F0A
-P 13950 3050
-F 0 "D44" H 13950 2833 50  0000 C CNN
-F 1 "B5819W" H 13950 2924 50  0000 C CNN
-F 2 "Diode_SMD:D_SOD-123" H 13950 3050 50  0001 C CNN
-F 3 "" H 13950 3050 50  0001 C CNN
-	1    13950 3050
-	-1   0    0    1
-$EndComp
 Wire Wire Line
 	14100 3050 14425 3050
@@
 Text Label 5775 9325 0    50   ~ 0
 PC12
+$Comp
+L micro_rusEFI-rescue:D_Schottky-Device D44
+U 1 1 618B2F0A
+P 13950 3050
+F 0 "D44" H 13950 2833 50  0000 C CNN
+F 1 "B5819W" H 13950 2924 50  0000 C CNN
+F 2 "Diode_SMD:D_SOD-123" H 13950 3050 50  0001 C CNN
+F 3 "" H 13950 3050 50  0001 C CNN
+	1    13950 3050
+	-1   0    0    1
+$EndComp
 $EndSCHEMATC

Commit message: Add files via upload
Parts:
- added unit 19 of U3
- D44: value B5819W -> 1N4148WS; footprint Diode_SMD:D_SOD-123 -> Diode_SMD:D_SOD-323
Connections:
- net CANH: now also U3.J49
- net CANL: now also U3.J50
Changed lines of the file:
@@
 Sheet 1 10
 Title "microRusEFI-2L"
-Date "2022-02-04"
+Date "2022-03-16"
 Rev "R0.5.5rc2"
 Comp "rusEFI.com"
 Comment1 "Donald Becker"
-Comment2 "AI6OD"
-Comment3 "by JRD McLAREN"
+Comment2 "by JRD McLAREN"
+Comment3 ""
 Comment4 ""
 $EndDescr
@@
 Text Label 11675 4225 0    60   ~ 12
 INJECTOR-4
-$Comp
-L micro_rusEFI-rescue:molex_48pin_MRE-rusefi_Molex_MRE_Connector U3
-U 1 1 5DD8BB43
-P 7750 2125
-F 0 "U3" V 9037 2530 60  0000 C CNN
-F 1 "molex_48pin_MRE" V 8931 2530 60  0000 C CNN
-F 2 "rusefi_lib:Molex_48_MRE_R055" H 7750 2125 60  0001 C CNN
-F 3 "" H 7750 2125 60  0001 C CNN
-F 4 "MOLEX" H 0   0   50  0001 C CNN "Manufacturer"
-F 5 "500762-0481" H 0   0   50  0001 C CNN "Part #"
-F 6 "DIGI" H 0   0   50  0001 C CNN "VEND"
-F 7 "WM4430-ND" H 0   0   50  0001 C CNN "VEND#"
-	1    7750 2125
-	0    -1   -1   0
-$EndComp
 Text Label 8350 1650 3    60   ~ 12
 GP2
@@
 $Comp
 L micro_rusEFI-rescue:molex_48pin_MRE-rusefi_Molex_MRE_Connector U3
-U 18 1 61B342CA
-P 11650 6400
-F 0 "U3" H 12578 6353 60  0000 L CNN
-F 1 "molex_48pin_MRE" V 12850 6400 60  0001 C CNN
-F 2 "rusefi_lib:Molex_48_MRE_R055" H 11650 6400 60  0001 C CNN
-F 3 "" H 11650 6400 60  0001 C CNN
-	18   11650 6400
-	1    0    0    -1
-$EndComp
-$Comp
-L micro_rusEFI-rescue:molex_48pin_MRE-rusefi_Molex_MRE_Connector U3
 U 17 1 61DBF805
 P 14225 3200
@@
 Wire Wire Line
 	14625 3350 14825 3350
-Wire Wire Line
-	12350 6350 12200 6350
-Wire Wire Line
-	12350 6500 12200 6500
-Text Label 12200 6350 2    50   ~ 10
-CANH
-Text Label 12200 6500 2    50   ~ 10
-CANL
 Text Label 6600 9225 2    50   ~ 0
 PC10
@@
 P 13950 3050
 F 0 "D44" H 13950 2833 50  0000 C CNN
-F 1 "B5819W" H 13950 2924 50  0000 C CNN
-F 2 "Diode_SMD:D_SOD-123" H 13950 3050 50  0001 C CNN
+F 1 "1N4148WS" H 13950 2924 50  0000 C CNN
+F 2 "Diode_SMD:D_SOD-323" H 13950 3050 50  0001 C CNN
 F 3 "" H 13950 3050 50  0001 C CNN
 	1    13950 3050
 	-1   0    0    1
 $EndComp
+Text Label 12200 6500 2    50   ~ 10
+CANL
+Text Label 12200 6350 2    50   ~ 10
+CANH
+Wire Wire Line
+	12350 6500 12200 6500
+Wire Wire Line
+	12350 6350 12200 6350
+$Comp
+L micro_rusEFI-rescue:molex_48pin_MRE-rusefi_Molex_MRE_Connector U3
+U 18 1 61B342CA
+P 11650 6400
+F 0 "U3" H 12578 6353 60  0000 L CNN
+F 1 "molex_48pin_MRE" V 12850 6400 60  0001 C CNN
+F 2 "rusefi_lib:Molex_48_MRE_R055" H 11650 6400 60  0001 C CNN
+F 3 "" H 11650 6400 60  0001 C CNN
+	18   11650 6400
+	1    0    0    -1
+$EndComp
+$Comp
+L micro_rusEFI-rescue:molex_48pin_MRE-rusefi_Molex_MRE_Connector U3
+U 1 1 5DD8BB43
+P 7750 2125
+F 0 "U3" V 9037 2530 60  0000 C CNN
+F 1 "molex_48pin_MRE" V 8931 2530 60  0000 C CNN
+F 2 "rusefi_lib:Molex_48_MRE_R055" H 7750 2125 60  0001 C CNN
+F 3 "" H 7750 2125 60  0001 C CNN
+F 4 "MOLEX" H 0   0   50  0001 C CNN "Manufacturer"
+F 5 "500762-0481" H 0   0   50  0001 C CNN "Part #"
+F 6 "DIGI" H 0   0   50  0001 C CNN "VEND"
+F 7 "WM4430-ND" H 0   0   50  0001 C CNN "VEND#"
+	1    7750 2125
+	0    -1   -1   0
+$EndComp
+Text Label 12200 6900 2    50   ~ 10
+CANL
+Text Label 12200 6750 2    50   ~ 10
+CANH
+Wire Wire Line
+	12350 6900 12200 6900
+Wire Wire Line
+	12350 6750 12200 6750
+$Comp
+L micro_rusEFI-rescue:molex_48pin_MRE-rusefi_Molex_MRE_Connector U3
+U 19 1 6244B367
+P 11650 6800
+F 0 "U3" H 12578 6753 60  0000 L CNN
+F 1 "molex_48pin_MRE" V 12850 6800 60  0001 C CNN
+F 2 "rusefi_lib:Molex_48_MRE_R055" H 11650 6800 60  0001 C CNN
+F 3 "" H 11650 6800 60  0001 C CNN
+	19   11650 6800
+	1    0    0    -1
+$EndComp
 $EndSCHEMATC
