File: TLE8888-1QK.sch (KiCad schematic (older format))
At the start: 40 parts, among them J15 Conn_01x01, J17 Conn_01x01, Q1 IPD30N06S2L-23, U2 TLE8888QK

Commit message: Add files via upload
Parts:
- C1, C10, C11, C12, C13, C14, C3, C35, C4, C41, C43, C5, C6, C7, C8, C9: symbol Device:C -> micro_rusEFI-rescue:C-Device
- C2: symbol Device:CP -> micro_rusEFI-rescue:CP-Device
- D1: symbol Diode:BAV70 -> micro_rusEFI-rescue:BAV70-Diode
- FID3, FID4: symbol Mechanical:Fiducial -> micro_rusEFI-rescue:Fiducial-Mechanical
- J15, J17: symbol Connector_Generic:Conn_01x01 -> micro_rusEFI-rescue:Conn_01x01-Connector_Generic
- Q1: symbol Transistor_FET:BUZ11 -> micro_rusEFI-rescue:BUZ11-Transistor_FET
- R12, R13, R15, R17, R18, R19, R20, R22, R3, R4, R6, R8, R82, R83, R9: symbol Device:R -> micro_rusEFI-rescue:R-Device
Changed lines of the file:
@@
 $Descr User 19685 15748
 encoding utf-8
-Sheet 8 9
+Sheet 7 10
 Title "microRusEFI-2L"
 Date "2020-05-24"
@@
 Connection ~ 6900 8600
 $Comp
-L Device:C C3
+L micro_rusEFI-rescue:C-Device C3
 U 1 1 5C5FD26E
 P 6900 8850
@@
 V5V
 $Comp
-L Device:C C10
+L micro_rusEFI-rescue:C-Device C10
 U 1 1 5C61E5D6
 P 10100 12050
@@
 $EndComp
 $Comp
-L power:GND #PWR015
+L micro_rusEFI-rescue:GND-power #PWR015
 U 1 1 5C620B15
 P 9600 11625
@@
 $EndComp
 $Comp
-L Device:CP C2
+L micro_rusEFI-rescue:CP-Device C2
 U 1 1 5C6EF1A0
 P 6200 8850
@@
 	5550 8600 5900 8600
 $Comp
-L Device:C C1
+L micro_rusEFI-rescue:C-Device C1
 U 1 1 5C6F613C
 P 5900 8850
@@
 	5900 9100 5900 9000
 $Comp
-L power:GND #PWR01
+L micro_rusEFI-rescue:GND-power #PWR01
 U 1 1 5C6FD38D
 P 5900 9100
@@
 	10100 11850 10100 11900
 $Comp
-L Device:C C11
+L micro_rusEFI-rescue:C-Device C11
 U 1 1 5C7331E3
 P 9600 11475
@@
 $EndComp
 $Comp
-L Device:C C4
+L micro_rusEFI-rescue:C-Device C4
 U 1 1 5C74BEC0
 P 8000 11800
@@
 $EndComp
 $Comp
-L Device:C C6
+L micro_rusEFI-rescue:C-Device C6
 U 1 1 5C758589
 P 8600 11800
@@
 $EndComp
 $Comp
-L Device:C C5
+L micro_rusEFI-rescue:C-Device C5
 U 1 1 5C760098
 P 8300 11850
@@
 	9350 10100 9350 10850
 $Comp
-L Device:C C7
+L micro_rusEFI-rescue:C-Device C7
 U 1 1 5C7776C3
 P 8900 11800
@@
 	11500 8150 11600 8150
 $Comp
-L Device:C C13
+L micro_rusEFI-rescue:C-Device C13
 U 1 1 5C7BB922
 P 12925 8375
@@
 OUT_18
 $Comp
-L Device:C C12
+L micro_rusEFI-rescue:C-Device C12
 U 1 1 5C88CC5C
 P 12000 6400
@@
 $EndComp
 $Comp
-L Device:R R12
+L micro_rusEFI-rescue:R-Device R12
 U 1 1 5C89FE8C
 P 12350 6250
@@
 $EndComp
 $Comp
-L Device:R R13
+L micro_rusEFI-rescue:R-Device R13
 U 1 1 5C8A058E
 P 12350 6550
@@
 $EndComp
 $Comp
-L Device:R R17
+L micro_rusEFI-rescue:R-Device R17
 U 1 1 5C8A0B54
 P 13075 5900
@@
 $EndComp
 $Comp
-L power:GND #PWR022
+L micro_rusEFI-rescue:GND-power #PWR022
 U 1 1 5C99C043
 P 15125 7600
@@
 OUT_21
 $Comp
-L power:GND #PWR06
+L micro_rusEFI-rescue:GND-power #PWR06
 U 1 1 5CA2A1BE
 P 8650 6600
@@
 $EndComp
 $Comp
-L power:GND #PWR016
+L micro_rusEFI-rescue:GND-power #PWR016
 U 1 1 5CA2C3D4
 P 11550 7250
@@
 OUT_23
 $Comp
-L power:GND #PWR03
+L micro_rusEFI-rescue:GND-power #PWR03
 U 1 1 5CB2A7FC
 P 8100 9600
@@
 	8100 8200 8000 8200
 $Comp
-L power:GND #PWR019
+L micro_rusEFI-rescue:GND-power #PWR019
 U 1 1 5CF6BD32
 P 11500 9650
@@
 	13025 7150 13175 7150
 $Comp
-L Device:C C14
+L micro_rusEFI-rescue:C-Device C14
 U 1 1 5D311D7B
 P 13025 7300
@@
 $EndComp
 $Comp
-L Device:R R20
+L micro_rusEFI-rescue:R-Device R20
 U 1 1 5D31001A
 P 13325 7150
@@
 Connection ~ 14325 7950
 $Comp
-L Device:R R6
+L micro_rusEFI-rescue:R-Device R6
 U 1 1 5D1AC4DC
 P 12000 7450
@@
 	11850 7450 11500 7450
 $Comp
-L Device:C C9
+L micro_rusEFI-rescue:C-Device C9
 U 1 1 5D1D1183
 P 9700 12050
@@
 	11500 9550 12225 9550
 $Comp
-L power:GND #PWR014
+L micro_rusEFI-rescue:GND-power #PWR014
 U 1 1 5C7B1869
 P 10950 10100
@@
 $EndComp
 $Comp
-L power:GND #PWR012
+L micro_rusEFI-rescue:GND-power #PWR012
 U 1 1 5C7C9FDD
 P 10350 10100
@@
 $EndComp
 $Comp
-L power:GND #PWR08
+L micro_rusEFI-rescue:GND-power #PWR08
 U 1 1 5C7CA872
 P 9050 10450
@@
 	9050 10100 9050 10450
 $Comp
-L power:GND #PWR011
+L micro_rusEFI-rescue:GND-power #PWR011
 U 1 1 5C7D9FD6
 P 10100 12200
@@
 $EndComp
 $Comp
-L power:GND #PWR010
+L micro_rusEFI-rescue:GND-power #PWR010
 U 1 1 5C7DA47B
 P 9700 12200
@@
 $EndComp
 $Comp
-L power:GND #PWR07
+L micro_rusEFI-rescue:GND-power #PWR07
 U 1 1 5C7DAF8E
 P 8900 11950
@@
 $EndComp
 $Comp
-L power:GND #PWR05
+L micro_rusEFI-rescue:GND-power #PWR05
 U 1 1 5C7DB5F1
 P 8600 11950
@@
 $EndComp
 $Comp
-L power:GND #PWR04
+L micro_rusEFI-rescue:GND-power #PWR04
 U 1 1 5C7DBB85
 P 8300 12000
@@
 $EndComp
 $Comp
-L power:GND #PWR02
+L micro_rusEFI-rescue:GND-power #PWR02
 U 1 1 5C7DC0D5
 P 8000 11950
@@
 	8000 10850 8000 11650
 $Comp
-L power:GND #PWR020
+L micro_rusEFI-rescue:GND-power #PWR020
 U 1 1 5C86C714
 P 12925 8525
@@
 $EndComp
 $Comp
-L power:GND #PWR021
+L micro_rusEFI-rescue:GND-power #PWR021
 U 1 1 5C86F645
 P 13300 7450
@@
 	7575 10300 8650 10300
 $Comp
-L Device:R R22
+L micro_rusEFI-rescue:R-Device R22
 U 1 1 5CEB6C29
 P 14200 7600
@@
 	13000 6700 13050 6700
 $Comp
-L Device:R R19
+L micro_rusEFI-rescue:R-Device R19
 U 1 1 5CC3675A
 P 13200 6700
@@
 $EndComp
 $Comp
-L Device:R R18
+L micro_rusEFI-rescue:R-Device R18
 U 1 1 5C8A82EA
 P 13200 6800
@@
 	9850 10100 10050 10100
 $Comp
-L Device:C C35
+L micro_rusEFI-rescue:C-Device C35
 U 1 1 5D394376
 P 12675 6400
@@
 $EndComp
 $Comp
-L Device:R R15
+L micro_rusEFI-rescue:R-Device R15
 U 1 1 5D394E3F
 P 12850 6400
@@
 	12725 6250 12850 6250
 $Comp
-L Mechanical:Fiducial FID3
+L micro_rusEFI-rescue:Fiducial-Mechanical FID3
 U 1 1 5D1D4069
 P 7300 6855
@@
 $EndComp
 $Comp
-L Mechanical:Fiducial FID4
+L micro_rusEFI-rescue:Fiducial-Mechanical FID4
 U 1 1 5D1D47C2
 P 7300 7050
@@
 Connection ~ 10650 5625
 $Comp
-L Device:C C43
+L micro_rusEFI-rescue:C-Device C43
 U 1 1 5D8748D4
 P 11250 5975
@@
 	10650 5625 10600 5625
 $Comp
-L power:GND #PWR0119
+L micro_rusEFI-rescue:GND-power #PWR0119
 U 1 1 5D8B9984
 P 11250 6125
@@
 	11500 7750 12000 7750
 $Comp
-L Device:C C41
+L micro_rusEFI-rescue:C-Device C41
 U 1 1 5E837BB7
 P 12150 7750
@@
 $EndComp
 $Comp
-L power:GND #PWR025
+L micro_rusEFI-rescue:GND-power #PWR025
 U 1 1 5E83818F
 P 12300 7750
@@
 12V_SAFE
 $Comp
-L power:PWR_FLAG #FLG0108
+L micro_rusEFI-rescue:PWR_FLAG-power #FLG0108
 U 1 1 5E9B7DD3
 P 12925 8150
@@
 $EndComp
 $Comp
-L Transistor_FET:BUZ11 Q1
+L micro_rusEFI-rescue:BUZ11-Transistor_FET Q1
 U 1 1 5C60C906
 P 10000 11450
@@
 	9350 11850 9350 11900
 $Comp
-L power:GND #PWR09
+L micro_rusEFI-rescue:GND-power #PWR09
 U 1 1 5C7DA925
 P 9350 12200
@@
 $EndComp
 $Comp
-L Device:C C8
+L micro_rusEFI-rescue:C-Device C8
 U 1 1 5D1F4F31
 P 9350 12050
@@
 	8100 7800 8000 7800
 $Comp
-L Diode:BAV70 D1
+L micro_rusEFI-rescue:BAV70-Diode D1
 U 1 1 5D872064
 P 11150 5625
@@
 	11050 6450 11900 6450
 $Comp
-L Device:R R8
+L micro_rusEFI-rescue:R-Device R8
 U 1 1 5E15579B
 P 11925 8050
@@
 INJ_EN
 $Comp
-L Device:R R82
+L micro_rusEFI-rescue:R-Device R82
 U 1 1 5E9E9D1E
 P 12225 9750
@@
 $EndComp
 $Comp
-L Device:R R83
+L micro_rusEFI-rescue:R-Device R83
 U 1 1 5E9F2CF7
 P 12225 10500
@@
 $EndComp
 $Comp
-L power:GND #PWR0113
+L micro_rusEFI-rescue:GND-power #PWR0113
 U 1 1 5EA00348
 P 12225 9950
@@
 $EndComp
 $Comp
-L power:GND #PWR0116
+L micro_rusEFI-rescue:GND-power #PWR0116
 U 1 1 5EA08CD1
 P 12225 10700
@@
 	7200 10700 9250 10700
 $Comp
-L Device:R R4
+L micro_rusEFI-rescue:R-Device R4
 U 1 1 5CC7AE36
 P 7425 9900
@@
 	7425 10050 7425 10150
 $Comp
-L Connector_Generic:Conn_01x01 J15
+L micro_rusEFI-rescue:Conn_01x01-Connector_Generic J15
 U 1 1 5EA3F4B2
 P 8100 6675
@@
 $EndComp
 $Comp
-L Connector_Generic:Conn_01x01 J17
+L micro_rusEFI-rescue:Conn_01x01-Connector_Generic J17
 U 1 1 5EA86A4A
 P 11500 10100
@@
 	8100 9850 8000 9850
 $Comp
-L Device:R R3
+L micro_rusEFI-rescue:R-Device R3
 U 1 1 5CC90402
 P 7425 10300
@@
 	12850 6200 12850 5575
 $Comp
-L Device:R R9
+L micro_rusEFI-rescue:R-Device R9
 U 1 1 5C89DF79
 P 12175 6400
