File: TLE9201SG.sch (KiCad schematic (older format))
At the start: 7 parts, among them U4 TLE9201SG

Commit message: Add files via upload
Parts:
- C15, C18, C19: symbol Device:C -> micro_rusEFI-rescue:C-Device
- R1, R16, R42: symbol Device:R -> micro_rusEFI-rescue:R-Device
Changed lines of the file:
@@
 $Descr A 11000 8500
 encoding utf-8
-Sheet 2 9
+Sheet 2 10
 Title "microRusEFI-2L"
 Date "2020-05-24"
@@
 	4675 3250 5325 3250
 $Comp
-L power:GND #PWR0109
+L micro_rusEFI-rescue:GND-power #PWR0109
 U 1 1 5DE49458
 P 5725 4025
@@
 	4825 3550 5325 3550
 $Comp
-L Device:C C15
+L micro_rusEFI-rescue:C-Device C15
 U 1 1 5DE4B24C
 P 4825 4150
@@
 $EndComp
 $Comp
-L Device:R R1
+L micro_rusEFI-rescue:R-Device R1
 U 1 1 5DE4B55B
 P 6475 4050
@@
 $EndComp
 $Comp
-L power:GND #PWR0110
+L micro_rusEFI-rescue:GND-power #PWR0110
 U 1 1 5DE4B957
 P 4825 4350
@@
 $EndComp
 $Comp
-L power:GND #PWR0161
+L micro_rusEFI-rescue:GND-power #PWR0161
 U 1 1 5E76AE52
 P 6475 2550
@@
 	6475 3350 6750 3350
 $Comp
-L Device:C C18
+L micro_rusEFI-rescue:C-Device C18
 U 1 1 5D324D41
 P 5025 4150
@@
 $EndComp
 $Comp
-L power:GND #PWR0189
+L micro_rusEFI-rescue:GND-power #PWR0189
 U 1 1 5D324D4B
 P 5025 4350
@@
 	5025 4000 5025 3350
 $Comp
-L Device:R R42
+L micro_rusEFI-rescue:R-Device R42
 U 1 1 5D02EEB5
 P 7100 4000
@@
 $EndComp
 $Comp
-L Device:C C19
+L micro_rusEFI-rescue:C-Device C19
 U 1 1 5D02EEB4
 P 7400 4000
@@
 	6475 3250 6125 3250
 $Comp
-L Device:R R16
+L micro_rusEFI-rescue:R-Device R16
 U 1 1 5D2D1AE3
 P 6475 2775
