File: adc.sch (KiCad schematic (older format))
At the start: 87 parts, among them U35 MCP6004, U36 MCP6004, U46 MCP6004, U8 MCP6004

Commit message: Add files via upload
Parts:
- removed C16, C45, C46, C47, C48, C49, C50, C51, C52, C53, C54, C55, C56, C57, C58, C59: 100nF, Capacitor_SMD:C_0402_1005Metric, symbol Device:C
- added CN1, CN2, CN3, CN4: 100nF, Resistor_SMD:R_Array_Convex_4x0603, symbol micro_rusEFI-rescue:C_Pack04-Device
- C40, C79, C80, C82: symbol Device:C -> micro_rusEFI-rescue:C-Device
- D13, D38, D39, D40: symbol Power_Protection:NUP4202 -> micro_rusEFI-rescue:NUP4202-Power_Protection
- D29: symbol Device:LED -> micro_rusEFI-rescue:LED-Device
- FID5, FID6: symbol Mechanical:Fiducial -> micro_rusEFI-rescue:Fiducial-Mechanical
- R11, R131, R139, R14, R141, R23, R24, R25, R26, R27, R28, R31, R32, R34, R35, R37, R38, R39, R40, R41, R44, R46, R5, R52, R53, R54, R55, R56, R57, R58, R59, R60, R61, R62, R63, R64, R65, R66, R67, R68, R69, R7, R70, R71, R72, R73, R74, R75, R76, R77, R78, R79: symbol Device:R -> micro_rusEFI-rescue:R-Device
- RN13, RN2, RN3, RN4: symbol Device:R_Pack04 -> micro_rusEFI-rescue:R_Pack04-Device
- U35, U36, U46, U8: symbol Amplifier_Operational:MCP6004 -> micro_rusEFI-rescue:MCP6004-Amplifier_Operational
