File: hi-lo.sch (KiCad schematic (older format))
At the start: 14 parts, among them U31 MIC4427, U32 MIC4427, U33 MIC4427

Commit message: Add files via upload
Parts:
- C17, C78: symbol Device:C -> micro_rusEFI-rescue:C-Device
- JP2: symbol Jumper:SolderJumper_3_Open -> micro_rusEFI-rescue:SolderJumper_3_Open-Jumper
- R120, R121, R122, R123, R124, R125: symbol Device:R -> micro_rusEFI-rescue:R-Device
- RN5, RN6: symbol Device:R_Pack04 -> micro_rusEFI-rescue:R_Pack04-Device
- U31, U32, U33: symbol Driver_FET:MIC4427 -> micro_rusEFI-rescue:MIC4427-Driver_FET
Changed lines of the file:
@@
 $Descr B 17000 11000
 encoding utf-8
-Sheet 6 9
+Sheet 6 10
 Title "microRusEFI-2L"
 Date "2020-05-24"
@@
 	5750 8100 6150 8100
 $Comp
-L power:GND #PWR0153
+L micro_rusEFI-rescue:GND-power #PWR0153
 U 1 1 5D14AE1C
 P 5900 8800
@@
 Connection ~ 5950 6900
 $Comp
-L Device:C C78
+L micro_rusEFI-rescue:C-Device C78
 U 1 1 5D15752C
 P 4600 6550
@@
 $EndComp
 $Comp
-L power:GND #PWR0149
+L micro_rusEFI-rescue:GND-power #PWR0149
 U 1 1 5D157536
 P 4600 6750
@@
 $EndComp
 $Comp
-L Device:R R120
+L micro_rusEFI-rescue:R-Device R120
 U 1 1 5D157560
 P 7550 5350
@@
 $EndComp
 $Comp
-L power:GND #PWR0158
+L micro_rusEFI-rescue:GND-power #PWR0158
 U 1 1 5D157576
 P 6375 5925
@@
 	5650 5550 5975 5550
 $Comp
-L power:GND #PWR0150
+L micro_rusEFI-rescue:GND-power #PWR0150
 U 1 1 5D1575C4
 P 5950 6175
@@
 Ign4_MCU
 $Comp
-L Device:C C17
+L micro_rusEFI-rescue:C-Device C17
 U 1 1 5E89211D
 P 4000 5200
@@
 $EndComp
 $Comp
-L power:GND #PWR0164
+L micro_rusEFI-rescue:GND-power #PWR0164
 U 1 1 5E892127
 P 4000 5425
@@
 12V
 $Comp
-L Device:R R121
+L micro_rusEFI-rescue:R-Device R121
 U 1 1 5D8F7DF1
 P 7550 5550
@@
 $EndComp
 $Comp
-L Device:R R122
+L micro_rusEFI-rescue:R-Device R122
 U 1 1 5D8F8794
 P 7600 6700
@@
 $EndComp
 $Comp
-L Device:R R124
+L micro_rusEFI-rescue:R-Device R124
 U 1 1 5D8FA32D
 P 7650 7900
@@
 $EndComp
 $Comp
-L Device:R R125
+L micro_rusEFI-rescue:R-Device R125
 U 1 1 5D8FA880
 P 7650 8100
@@
 $EndComp
 $Comp
-L Device:R R123
+L micro_rusEFI-rescue:R-Device R123
 U 1 1 5D8F9107
 P 7600 6900
@@
 $EndComp
 $Comp
-L Jumper:SolderJumper_3_Open JP2
+L micro_rusEFI-rescue:SolderJumper_3_Open-Jumper JP2
 U 1 1 5DAB9BDF
 P 3550 4800
@@
 	3550 4950 3550 5050
 $Comp
-L Device:R_Pack04 RN5
+L micro_rusEFI-rescue:R_Pack04-Device RN5
 U 1 1 5DB3A3BD
 P 5950 8500
@@
 	5950 8700 6050 8700
 $Comp
-L Device:R_Pack04 RN6
+L micro_rusEFI-rescue:R_Pack04-Device RN6
 U 1 1 5DB70BD2
 P 5850 5975
@@
 NoConn ~ 5950 5775
 $Comp
-L Driver_FET:MIC4427 U31
+L micro_rusEFI-rescue:MIC4427-Driver_FET U31
 U 1 1 5DB97186
 P 6375 5450
@@
 5V
 $Comp
-L Driver_FET:MIC4427 U33
+L micro_rusEFI-rescue:MIC4427-Driver_FET U33
 U 1 1 5DBA9C1F
 P 6550 8000
@@
 $EndComp
 $Comp
-L power:GND #PWR0137
+L micro_rusEFI-rescue:GND-power #PWR0137
 U 1 1 5DBAA76F
 P 6550 8450
@@
 $EndComp
 $Comp
-L Driver_FET:MIC4427 U32
+L micro_rusEFI-rescue:MIC4427-Driver_FET U32
 U 1 1 5DBAB8DF
 P 6500 6800
@@
 $EndComp
 $Comp
-L power:GND #PWR0146
+L micro_rusEFI-rescue:GND-power #PWR0146
 U 1 1 5DBABE2E
 P 6500 7250
@@
 Connection ~ 6500 6400
 $Comp
-L power:PWR_FLAG #FLG0107
+L micro_rusEFI-rescue:PWR_FLAG-power #FLG0107
 U 1 1 5DBBE02C
 P 3550 5050
