File: pair.sch (KiCad schematic (older format))
At the start: 1 part, among them U1 VNLD5090

Commit message: Add files via upload
Changed lines of the file:
@@
 $Descr A4 11693 8268
 encoding utf-8
-Sheet 4 9
+Sheet 4 10
 Title "microRusEFI-2L"
 Date "2020-05-24"
@@
 $EndComp
 $Comp
-L power:GND #PWR0113
+L micro_rusEFI-rescue:GND-power #PWR0113
 U 1 1 5E290D55
 P 3300 2500
@@
 $EndComp
 $Comp
-L power:GND #PWR0114
+L micro_rusEFI-rescue:GND-power #PWR0114
 U 1 1 5E291066
 P 3400 2500
