File: stm32.sch (KiCad schematic (older format))
At the start: 47 parts, among them J1 USB_B_Micro, J19 Conn_01x06, J2 Conn_02x05_Odd_Even, J7 TC2030, SW1 SW_Push, SW2 SW_Push, SW3 SW_Push, SW4 SW_Push, U1 STM32F427VGT6, U3 molex_48pin_MRE, U5 LM1117-3.3, X1 8MHz 20pF, Y2 32768 Hz

Commit message: Add files via upload
Parts:
- C20, C21, C22, C23, C24, C25, C26, C27, C28, C29, C30, C31, C32, C33, C34, C36, C37, C38, C39, C44: symbol Device:C -> micro_rusEFI-rescue:C-Device
- D14: footprint Capacitor_SMD:C_0805_2012Metric -> LED_SMD:LED_0603_1608Metric; symbol Device:LED -> micro_rusEFI-rescue:LED-Device
- D16: symbol Power_Protection:NUP4202 -> micro_rusEFI-rescue:NUP4202-Power_Protection
- D17: symbol Device:D_Schottky -> micro_rusEFI-rescue:D_Schottky-Device
- D19: symbol Device:LED -> micro_rusEFI-rescue:LED-Device
- D42: symbol Diode:BAV70 -> micro_rusEFI-rescue:BAV70-Diode
- FB1: symbol Device:Ferrite_Bead -> micro_rusEFI-rescue:Ferrite_Bead-Device
- FID1, FID2: symbol Mechanical:Fiducial -> micro_rusEFI-rescue:Fiducial-Mechanical
- J1: symbol Connector:USB_B_Micro -> micro_rusEFI-rescue:USB_B_Micro-Connector
- J19: symbol Connector_Generic:Conn_01x05 -> micro_rusEFI-rescue:Conn_01x05-Connector_Generic
- J2: symbol Connector_Generic:Conn_02x05_Odd_Even -> micro_rusEFI-rescue:Conn_02x05_Odd_Even-Connector_Generic
- J7: symbol Connector:Conn_01x06_Male -> micro_rusEFI-rescue:Conn_01x06_Male-Connector
- NT1: symbol Device:Net-Tie_2 -> micro_rusEFI-rescue:Net-Tie_2-Device
- R43, R45, R47, R48, R50: symbol Device:R -> micro_rusEFI-rescue:R-Device
- SW1, SW2, SW3, SW4: symbol Switch:SW_Push -> micro_rusEFI-rescue:SW_Push-Switch
- U1: symbol MCU_ST_STM32F4:STM32F407VGTx -> micro_rusEFI-rescue:STM32F407VGTx-MCU_ST_STM32F4
- U3: footprint (none) -> rusefi_lib:Molex_48_MRE_R055; symbol rusefi_Molex_MRE_Connector:molex_48pin_MRE -> micro_rusEFI-rescue:molex_48pin_MRE-rusefi_Molex_MRE_Connector
- U5: symbol Regulator_Linear:LM1117-3.3 -> micro_rusEFI-rescue:LM1117-3.3-Regulator_Linear
- X1: symbol Device:Crystal -> micro_rusEFI-rescue:Crystal-Device
- Y2: symbol Device:Crystal_Small -> micro_rusEFI-rescue:Crystal_Small-Device

Commit message: Add files via upload
Parts:
- C39: footprint Capacitor_SMD:C_0603_1608Metric -> Capacitor_SMD:C_0805_2012Metric
Changed lines of the file:
@@
 Sheet 9 10
 Title "microRusEFI-2L"
-Date "2020-05-24"
-Rev "R0.5.2"
+Date "2021-11-11"
+Rev "R0.5.5rc"
 Comp "rusEFI.com"
 Comment1 "Donald Becker"
@@
 F 0 "C39" H 15450 3000 50  0000 C CNN
 F 1 "22uF" H 15450 2800 50  0000 C CNN
-F 2 "Capacitor_SMD:C_0603_1608Metric" V 11930 4200 60  0001 C CNN
+F 2 "Capacitor_SMD:C_0805_2012Metric" V 11930 4200 60  0001 C CNN
 F 3 "" H 15350 2900 60  0001 C CNN
 F 4 "stm32f407_board" H 23450 3775 60  0001 C CNN "PageName"
