File: micro_rusEFI.kicad_pcb (KiCad board)
At the start: 2 copper layers, 80.6 x 93.7 mm, 246 parts, among them CN1 100nF, CN2 100nF, CN3 100nF, CN4 100nF, J1 USB_B_Micro, J12 Conn_01x01, J13 Conn_01x01, J14 microSD_HC_Wuerth_693072010801, J15 Conn_01x01, J17 Conn_01x01, J19 Conn_01x06, J2 Conn_02x05_Odd_Even, J3 Conn_01x01, J4 Conn_02x05_Counter_Clockwise, J5 Conn_01x01, J7 TC2030, Q1 IPD30N06S2L-23, SW1 SW_Push, SW2 SW_Push, SW3 SW_Push, SW4 SW_Push, U1 STM32F427VGT6, U10 VNLD5090, U2 TLE8888QK, U3 molex_48pin_MRE, U31 MIC4427, U32 MIC4427, U33 MIC4427, U35 MCP6004, U36 MCP6004, U4 TLE9201SG, U46 MCP6004, U5 LM1117-3.3, U6 W25Q128JVSIQ, U7 XC6206 3.3V, U8 MCP6004, U9 VNLD5090, X1 8MHz 20pF, Y2 32768 Hz

Commit message: Add files via upload
Parts:
- moved J3 12.2 mm to (41.2, 24.1), turned to 0 degrees
- moved D34 12.0 mm to (23.1, 35.1)
- moved J5 9.53 mm to (37.7, 24.1)
- moved D6 6.72 mm to (30.7, 28.5), turned to 90 degrees
- moved J13 4.90 mm to (34.2, 24.1)
- moved D3 3.30 mm to (37.7, 28.5), turned to 90 degrees
- moved D4 2.74 mm to (41.2, 28.5), turned to 90 degrees
- moved D5 1.76 mm to (34.2, 28.5), turned to 90 degrees
- moved R51 1.62 mm to (26.3, 35.1), turned to 270 degrees
- moved D35 1.40 mm to (24.9, 35.1)
- moved D20 0.73 mm to (90.2, 26.7)
- moved D15 0.71 mm to (92.0, 29.9)
- moved J12 0.10 mm to (30.7, 24.1)
Routing:
- net GND: track 126.7 -> 149.7 mm, vias 518 -> 517
- net /12V_MREL: track 282.8 -> 269.7 mm
- net /5V: track 474.0 -> 485.8 mm
- net Net-(D34-Pad1): track 12.0 -> 2.58 mm
- net /GP5: track 64.5 -> 60.6 mm
- net /LS2: track 106.8 -> 108.1 mm
- net Net-(D3-Pad2): track 3.16 -> 2.50 mm
- net Net-(D35-Pad1): track 2.12 -> 1.50 mm
- net Net-(D4-Pad2): track 3.08 -> 2.50 mm

Commit message: Add files via upload
Parts:
- R131, R24, R31, R34, R37, R41, R52, R54, R56, R58: footprint Resistor_SMD:R_0402_1005Metric -> Resistor_SMD:R_0603_1608Metric
- moved R28 31.3 mm to (46.2, 45.1), turned to 270 degrees
- moved R34 10.8 mm to (70.2, 44.0), turned to 0 degrees
- moved R31 10.1 mm to (63.5, 40.9)
- moved R56 8.65 mm to (66.8, 39.4), turned to 0 degrees
- moved R58 8.07 mm to (70.2, 42.5)
- moved R24 7.65 mm to (66.8, 40.9), turned to 0 degrees
- moved R131 6.41 mm to (56.1, 39.4), turned to 0 degrees
- moved R37 6.05 mm to (63.5, 39.4), turned to 0 degrees
- moved R7 5.98 mm to (69.9, 45.4), turned to 180 degrees
- moved R41 5.50 mm to (56.1, 40.9), turned to 180 degrees
- moved R52 5.37 mm to (70.2, 40.9), turned to 0 degrees
- moved R11 4.82 mm to (51.9, 40.6), turned to 90 degrees
- moved CN4 3.56 mm to (62.2, 46.9)
- moved RN4 3.54 mm to (62.2, 43.3)
- moved RN2 3.54 mm to (66.8, 43.3)
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Routing:
- net /CAM_SENSOR: track 80.6 -> 29.7 mm
- net Net-(D29-Pad1): track 1.51 -> 41.6 mm
- net Net-(CN2-Pad2): track 33.7 -> 27.0 mm
- net /5V: track 485.8 -> 479.7 mm, vias 28 -> 30
- net /AV8: track 44.0 -> 49.0 mm, vias 1 -> 2
- net Net-(CN2-Pad4): track 26.7 -> 22.3 mm
- net /AV3: track 6.74 -> 10.8 mm
- net /AV10: track 52.8 -> 56.9 mm, vias 1 -> 4
- net /AV1: track 7.15 -> 11.1 mm
- net /AV2: track 8.89 -> 12.7 mm
- net Net-(CN2-Pad3): track 29.6 -> 25.8 mm
- net Net-(CN2-Pad1): track 29.2 -> 25.6 mm
- net Net-(CN4-Pad5): track 18.8 -> 15.3 mm
- net Net-(CN4-Pad7): track 21.3 -> 18.1 mm
- net Net-(CN4-Pad8): track 17.9 -> 14.9 mm
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Other:
- board text added: "microRusEFI R0.5.5rc2"
