File: micro_rusEFI.kicad_pcb (KiCad board)
At the start: 2 copper layers, 80.6 x 93.7 mm, 250 parts, among them CN1 100nF, CN2 100nF, CN3 100nF, CN4 100nF, J1 USB_B_Micro, J12 Conn_01x01, J13 Conn_01x01, J14 microSD_HC_Wuerth_693072010801, J15 Conn_01x01, J17 Conn_01x01, J19 Conn_01x06, J2 Conn_02x05_Odd_Even, J3 Conn_01x01, J4 Conn_02x05_Counter_Clockwise, J5 Conn_01x01, J7 TC2030, Q1 IPD30N06S2L-23, SW1 SW_Push, SW2 SW_Push, SW3 SW_Push, SW4 SW_Push, U1 STM32F427VGT6, U10 VNLD5090, U2 TLE8888QK, U3 molex_48pin_MRE, U31 MIC4427, U32 MIC4427, U33 MIC4427, U35 MCP6004, U36 MCP6004, U4 TLE9201SG, U46 MCP6004, U5 LM1117-3.3, U6 W25Q128JVSIQ, U7 XC6206 3.3V, U8 MCP6004, U9 VNLD5090, X1 8MHz 20pF, Y2 32768 Hz

Commit message: Add files via upload
Parts:
- D44: value B5819W -> 1N4148WS; footprint Diode_SMD:D_SOD-123 -> Diode_SMD:D_SOD-323
- moved J14 0.22 mm to (76.0, 108.2)
- moved J19 0.10 mm to (59.6, 97.5)
- moved C27 0.06 mm to (71.5, 93.8)
- moved C29 0.06 mm to (69.9, 93.8)
- moved C23 0.05 mm to (66.3, 93.8)
- moved C24 0.05 mm to (67.8, 93.8)
Routing:
- net GND: track 151.1 -> 148.4 mm, vias 472 -> 470
- net Net-(D44-Pad1): track 11.0 -> 11.7 mm
- net /VDD: track 351.8 -> 352.1 mm, vias 32 -> 33
- net /MCU/PB15: vias 2 -> 3
Other:
- outline, holes or cut-outs redrawn

Commit message: Add files via upload
Routing:
- net /PB9: track 102.2 -> 103.1 mm
- net GND: vias 470 -> 472
- net /VDD: vias 33 -> 32
- net /MCU/PB15: vias 3 -> 2
